Commit message: Added Lidar in gazebo

File: qhali_description/urdf/qhali.xacro (robot description, xacro)
@@ -3,5 +3,7 @@
 <xacro:include filename="$(find qhali_description)/urdf/materials.xacro" />
 <xacro:include filename="$(find qhali_description)/urdf/qhali.trans" />
-<xacro:include filename="$(find qhali_description)/urdf/qhali.gazebo" />
+<xacro:include filename="$(find qhali_description)/gazebo/qhali_materials.gazebo" />
+<xacro:include filename="$(find qhali_description)/gazebo/qhali_physics.gazebo" />
+<xacro:include filename="$(find qhali_description)/gazebo/qhali_plugins.gazebo" />
 <link name="base_link">
   <inertial>
@@ -981,4 +983,24 @@
     <geometry>
       <mesh filename="package://qhali_description/meshes/right_skirt_sblue_case_link_1.stl" scale="0.001 0.001 0.001"/>
+    </geometry>
+  </collision>
+</link>
+<link name="rplidar">
+  <inertial>
+    <origin xyz="0.0 0.0 0.0205" rpy="0 0 0"/>
+    <mass value="0.19"/>
+    <inertia ixx="1e-5" iyy="1e-5" izz="1e-5" ixy="0" iyz="0" ixz="0"/>
+  </inertial>
+  <visual>
+    <origin xyz="0.0 0.0 0.0205" rpy="0 0 0"/>
+    <geometry>
+      <cylinder length="0.041" radius="0.038"/>
+    </geometry>
+    <material name="silver"/>
+  </visual>
+  <collision>
+    <origin xyz="0.0 0.0 0.0205" rpy="0 0 0"/>
+    <geometry>
+      <cylinder length="0.041" radius="0.038"/>
     </geometry>
   </collision>
@@ -998,5 +1020,5 @@
   <parent link="left_motor_link_1"/>
   <child link="left_wheel_link_1"/>
-  <axis xyz="-0.0 -1.0 -0.0"/>
+  <axis xyz="0.0 1.0 0.0"/>
 </joint>
 <joint name="front_right_caster_joint" type="fixed">
@@ -1024,5 +1046,5 @@
   <parent link="right_motor_link_1"/>
   <child link="right_wheel_link_1"/>
-  <axis xyz="0.0 -1.0 -0.0"/>
+  <axis xyz="0.0 1.0 0.0"/>
 </joint>
 <joint name="columns_joint" type="fixed">
@@ -1226,3 +1248,8 @@
   <child link="right_skirt_sblue_case_link_1"/>
 </joint>
+<joint name="lidar_joint" type="fixed">
+  <origin xyz="0.0 0.0 0.0" rpy="0.0 0.0 0.0"/>
+  <parent link="mdf_link_1"/>
+  <child link="rplidar"/>
+</joint>
 </robot>

Commit message: Fixed lidar position

File: qhali_description/urdf/qhali.xacro (robot description, xacro)
@@ -988,10 +988,10 @@
 <link name="rplidar">
   <inertial>
-    <origin xyz="0.0 0.0 0.0205" rpy="0 0 0"/>
+    <origin xyz="0.0 0.0 -0.0205" rpy="0 0 0"/>
     <mass value="0.19"/>
     <inertia ixx="1e-5" iyy="1e-5" izz="1e-5" ixy="0" iyz="0" ixz="0"/>
   </inertial>
   <visual>
-    <origin xyz="0.0 0.0 0.0205" rpy="0 0 0"/>
+    <origin xyz="0.0 0.0 -0.0205" rpy="0 0 0"/>
     <geometry>
       <cylinder length="0.041" radius="0.038"/>
@@ -1000,5 +1000,5 @@
   </visual>
   <collision>
-    <origin xyz="0.0 0.0 0.0205" rpy="0 0 0"/>
+    <origin xyz="0.0 0.0 -0.0205" rpy="0 0 0"/>
     <geometry>
       <cylinder length="0.041" radius="0.038"/>
@@ -1249,5 +1249,6 @@
 </joint>
 <joint name="lidar_joint" type="fixed">
-  <origin xyz="0.0 0.0 0.0" rpy="0.0 0.0 0.0"/>
+  <!--Lidar beam height 3+41-->
+  <origin xyz="-0.020025 0.231825 0.044" rpy="0.0 0.0 0.0"/>
   <parent link="mdf_link_1"/>
   <child link="rplidar"/>

Commit message: Height of Lidar fixed

File: qhali_description/urdf/qhali.xacro (robot description, xacro)
@@ -988,10 +988,10 @@
 <link name="rplidar">
   <inertial>
-    <origin xyz="0.0 0.0 -0.0205" rpy="0 0 0"/>
+    <origin xyz="0.0 0.0 -0.0105" rpy="0 0 0"/>
     <mass value="0.19"/>
     <inertia ixx="1e-5" iyy="1e-5" izz="1e-5" ixy="0" iyz="0" ixz="0"/>
   </inertial>
   <visual>
-    <origin xyz="0.0 0.0 -0.0205" rpy="0 0 0"/>
+    <origin xyz="0.0 0.0 -0.0105" rpy="0 0 0"/>
     <geometry>
       <cylinder length="0.041" radius="0.038"/>
@@ -1000,5 +1000,5 @@
   </visual>
   <collision>
-    <origin xyz="0.0 0.0 -0.0205" rpy="0 0 0"/>
+    <origin xyz="0.0 0.0 -0.0105" rpy="0 0 0"/>
     <geometry>
       <cylinder length="0.041" radius="0.038"/>
@@ -1249,6 +1249,6 @@
 </joint>
 <joint name="lidar_joint" type="fixed">
-  <!--Lidar beam height 3+41-->
-  <origin xyz="-0.020025 0.231825 0.044" rpy="0.0 0.0 0.0"/>
+  <!--Lidar beam height 3+41+4-10-->
+  <origin xyz="-0.020025 0.231825 0.038" rpy="0.0 0.0 0.0"/>
   <parent link="mdf_link_1"/>
   <child link="rplidar"/>

Commit message: Added depth camera

File: qhali_description/urdf/qhali.xacro (robot description, xacro)
@@ -986,5 +986,5 @@
   </collision>
 </link>
-<link name="rplidar">
+<link name="rplidar_link">
   <inertial>
     <origin xyz="0.0 0.0 -0.0105" rpy="0 0 0"/>
@@ -1003,4 +1003,24 @@
     <geometry>
       <cylinder length="0.041" radius="0.038"/>
+    </geometry>
+  </collision>
+</link>
+<link name="depth_camera_link">
+  <inertial>
+    <origin xyz="0.0 0.0 0.0" rpy="0 1.57 0"/>
+    <mass value="0.095"/>
+    <inertia ixx="1e-5" iyy="1e-5" izz="1e-5" ixy="0" iyz="0" ixz="0"/>
+  </inertial>
+  <visual>
+    <origin xyz="0.0 0.0 0.0" rpy="0 1.57 0"/>
+    <geometry>
+      <cylinder length="0.026" radius="0.0305"/>
+    </geometry>
+    <material name="silver"/>
+  </visual>
+  <collision>
+    <origin xyz="0.0 0.0 0.0" rpy="0 1.57 0"/>
+    <geometry>
+      <cylinder length="0.026" radius="0.0305"/>
     </geometry>
   </collision>
@@ -1252,5 +1272,21 @@
   <origin xyz="-0.020025 0.231825 0.038" rpy="0.0 0.0 0.0"/>
   <parent link="mdf_link_1"/>
-  <child link="rplidar"/>
+  <child link="rplidar_link"/>
+</joint>
+<joint name="depth_joint" type="fixed">
+  <!--Lidar beam height 3+41+4-10-->
+  <origin xyz="0.47024 0.0 0.154026" rpy="0.0 0.0 0.0"/>
+  <parent link="skirt_white_case_link_1"/>
+  <child link="depth_camera_link"/>
+</joint>
+<link name="depth_camera_link_optical">
+</link>
+<joint name="depth_camera_optical_joint" type="fixed">
+  <!-- these values have to be these values otherwise the gazebo camera
+      image won't be aligned properly with the frame it is supposedly
+      originating from -->
+  <origin xyz="0 0 0" rpy="${-pi/2} 0 ${-pi/2}"/>
+  <parent link="depth_camera_link"/>
+  <child link="depth_camera_link_optical"/>
 </joint>
 </robot>

Commit message: Fixed depth camera position

File: qhali_description/urdf/qhali.xacro (robot description, xacro)
@@ -1008,10 +1008,10 @@
 <link name="depth_camera_link">
   <inertial>
-    <origin xyz="0.0 0.0 0.0" rpy="0 1.57 0"/>
+    <origin xyz="-0.0085 0.0 0.0" rpy="0 1.57 0"/>
     <mass value="0.095"/>
     <inertia ixx="1e-5" iyy="1e-5" izz="1e-5" ixy="0" iyz="0" ixz="0"/>
   </inertial>
   <visual>
-    <origin xyz="0.0 0.0 0.0" rpy="0 1.57 0"/>
+    <origin xyz="-0.0085 0.0 0.0" rpy="0 1.57 0"/>
     <geometry>
       <cylinder length="0.026" radius="0.0305"/>
@@ -1020,5 +1020,5 @@
   </visual>
   <collision>
-    <origin xyz="0.0 0.0 0.0" rpy="0 1.57 0"/>
+    <origin xyz="-0.0085 0.0 0.0" rpy="0 1.57 0"/>
     <geometry>
       <cylinder length="0.026" radius="0.0305"/>
